File: echo.brd (EAGLE design)
At the start: 99 x 50.5 mm, 109 parts, among them IC1 78L05Z, IC2 PT2399, IC3 TL074P, IC4 TL074P, IC5 LM13700N

Commit message: Add files via upload
Parts:
- C27, C28: device rcl:C050-055X075 -> rcl:C050-075X075
- moved R16 2.29 mm to (51.4, 34.9), turned to 270 degrees
Routing:
- net -12V: track 152.9 -> 151.7 mm
- net +12V: track 232.2 -> 231.5 mm
- added copper zone on layer 1, net GND
Other:
- board text added: "VC Echo"
Changed lines of the file:
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@@
 <wire x1="99.04" y1="50.47" x2="0" y2="50.47" width="0" layer="20"/>
 <wire x1="0" y1="50.47" x2="0" y2="0" width="0" layer="20"/>
+<text x="90.17" y="40.64" size="2.54" layer="21">VC
+Echo</text>
 </plain>
 <attributes>
@@
 <attribute name="VALUE" x="89.281" y="33.3248" size="1.27" layer="27" ratio="10" rot="R180"/>
 </element>
-<element name="R16" library="rcl" package="0309V" value="1M" x="52.705" y="36.83" smashed="yes">
-<attribute name="NAME" x="52.324" y="34.671" size="1.27" layer="25" ratio="10"/>
-<attribute name="VALUE" x="52.959" y="34.6202" size="1.27" layer="27" ratio="10"/>
+<element name="R16" library="rcl" package="0309V" value="1M" x="51.435" y="34.925" smashed="yes" rot="R270">
+<attribute name="NAME" x="49.276" y="35.306" size="1.27" layer="25" ratio="10" rot="R270"/>
+<attribute name="VALUE" x="49.2252" y="34.671" size="1.27" layer="27" ratio="10" rot="R270"/>
 </element>
 <element name="R17" library="rcl" package="0309V" value="3k" x="59.69" y="31.75" smashed="yes">
@@
 </element>
 <element name="R23" library="rcl" package="0309V" value="100k" x="57.15" y="47.625" smashed="yes" rot="R180">
-<attribute name="NAME" x="56.896" y="46.609" size="1.27" layer="25" ratio="10" rot="R180"/>
+<attribute name="NAME" x="58.166" y="49.784" size="1.27" layer="25" ratio="10" rot="R180"/>
 <attribute name="VALUE" x="56.896" y="49.8348" size="1.27" layer="27" ratio="10" rot="R180"/>
 </element>
@@
 <attribute name="VALUE" x="43.434" y="40.132" size="1.27" layer="27" ratio="10" rot="R270"/>
 </element>
-<element name="C28" library="rcl" package="C050-055X075" value="10u" x="53.34" y="41.91" smashed="yes">
-<attribute name="NAME" x="49.911" y="45.085" size="1.27" layer="25" ratio="10"/>
+<element name="C28" library="rcl" package="C050-075X075" value="10u" x="53.34" y="41.91" smashed="yes">
+<attribute name="NAME" x="49.53" y="41.656" size="1.27" layer="25" ratio="10" rot="R90"/>
 <attribute name="VALUE" x="50.038" y="39.624" size="1.27" layer="27" ratio="10"/>
 </element>
@@
 <attribute name="VALUE" x="86.614" y="33.909" size="1.27" layer="27" ratio="10" rot="R90"/>
 </element>
-<element name="C27" library="rcl" package="C050-055X075" value="10u" x="88.9" y="20.955" smashed="yes" rot="R270">
+<element name="C27" library="rcl" package="C050-075X075" value="10u" x="88.9" y="20.955" smashed="yes" rot="R270">
 <attribute name="NAME" x="85.725" y="21.971" size="1.27" layer="25" ratio="10" rot="R90"/>
 <attribute name="VALUE" x="86.614" y="24.257" size="1.27" layer="27" ratio="10" rot="R270"/>
@@
 <polygon width="0.4064" layer="16" isolate="0.8128" thermals="no">
 <vertex x="0" y="50.165"/>
-<vertex x="0" y="-0.635"/>
-<vertex x="99.06" y="-0.635"/>
+<vertex x="0" y="0"/>
+<vertex x="99.06" y="0"/>
 <vertex x="99.06" y="50.165"/>
+</polygon>
+<polygon width="0.4064" layer="1" isolate="0.6096" thermals="no">
+<vertex x="0.635" y="50.165"/>
+<vertex x="0.635" y="0"/>
+<vertex x="98.425" y="0"/>
+<vertex x="98.425" y="50.165"/>
 </polygon>
 </signal>
@@
 <wire x1="3.81" y1="19.05" x2="6.35" y2="19.05" width="0.6096" layer="16"/>
 <wire x1="6.35" y1="19.05" x2="11.43" y2="19.05" width="0.6096" layer="16"/>
-<wire x1="41.91" y1="38.735" x2="43.815" y2="36.83" width="0.6096" layer="16"/>
-<wire x1="43.815" y1="36.83" x2="51.435" y2="36.83" width="0.6096" layer="16"/>
+<wire x1="41.275" y1="38.735" x2="43.815" y2="36.195" width="0.6096" layer="16"/>
 <wire x1="35.56" y1="12.065" x2="32.385" y2="12.065" width="0.6096" layer="1"/>
 <wire x1="32.385" y1="12.065" x2="32.385" y2="10.795" width="0.6096" layer="1"/>
@@
 <wire x1="33.655" y1="20.955" x2="32.385" y2="19.685" width="0.6096" layer="1"/>
 <wire x1="32.385" y1="19.685" x2="32.385" y2="12.065" width="0.6096" layer="1"/>
-<wire x1="51.435" y1="36.83" x2="53.086" y2="35.179" width="0.6096" layer="1"/>
-<wire x1="53.086" y1="35.179" x2="59.055" y2="35.179" width="0.6096" layer="1"/>
 <wire x1="59.055" y1="35.179" x2="60.071" y2="36.195" width="0.6096" layer="1"/>
 <wire x1="60.071" y1="36.195" x2="60.071" y2="37.846" width="0.6096" layer="1"/>
@@
 <wire x1="76.2" y1="34.29" x2="76.2" y2="28.575" width="0.4064" layer="16"/>
 <wire x1="44.45" y1="31.115" x2="43.815" y2="31.75" width="0.6096" layer="16"/>
-<wire x1="43.815" y1="31.75" x2="43.815" y2="36.83" width="0.6096" layer="16"/>
+<wire x1="43.815" y1="31.75" x2="43.815" y2="36.195" width="0.6096" layer="16"/>
 <wire x1="31.75" y1="38.735" x2="33.02" y2="38.735" width="0.6096" layer="16"/>
 <wire x1="33.02" y1="38.735" x2="34.29" y2="40.005" width="0.6096" layer="16"/>
 <wire x1="34.29" y1="40.005" x2="36.83" y2="40.005" width="0.6096" layer="16"/>
 <wire x1="36.83" y1="40.005" x2="38.1" y2="38.735" width="0.6096" layer="16"/>
-<wire x1="38.1" y1="38.735" x2="41.91" y2="38.735" width="0.6096" layer="16"/>
+<wire x1="38.1" y1="38.735" x2="41.275" y2="38.735" width="0.6096" layer="16"/>
+<wire x1="43.815" y1="36.195" x2="51.435" y2="36.195" width="0.6096" layer="16"/>
+<wire x1="59.055" y1="35.179" x2="56.896" y2="35.179" width="0.6096" layer="1"/>
+<wire x1="56.896" y1="35.179" x2="55.88" y2="36.195" width="0.6096" layer="1"/>
+<wire x1="55.88" y1="36.195" x2="51.435" y2="36.195" width="0.6096" layer="1"/>
 </signal>
 <signal name="-12V">
@@
 <wire x1="27.305" y1="27.94" x2="27.305" y2="38.735" width="0.6096" layer="1"/>
 <wire x1="24.13" y1="38.735" x2="27.305" y2="38.735" width="0.6096" layer="1"/>
-<wire x1="41.91" y1="38.735" x2="43.815" y2="36.83" width="0.6096" layer="1"/>
-<wire x1="43.815" y1="36.83" x2="47.625" y2="36.83" width="0.6096" layer="1"/>
-<wire x1="47.625" y1="36.83" x2="49.53" y2="34.925" width="0.6096" layer="1"/>
-<wire x1="49.53" y1="34.925" x2="49.53" y2="31.115" width="0.6096" layer="1"/>
+<wire x1="41.275" y1="38.735" x2="43.18" y2="36.83" width="0.6096" layer="1"/>
 <wire x1="11.43" y1="27.94" x2="27.305" y2="27.94" width="0.6096" layer="1"/>
 <wire x1="27.305" y1="27.94" x2="28.575" y2="27.94" width="0.6096" layer="1"/>
@@
 <wire x1="33.655" y1="40.005" x2="36.83" y2="40.005" width="0.6096" layer="1"/>
 <wire x1="36.83" y1="40.005" x2="38.1" y2="38.735" width="0.6096" layer="1"/>
-<wire x1="38.1" y1="38.735" x2="41.91" y2="38.735" width="0.6096" layer="1"/>
+<wire x1="38.1" y1="38.735" x2="41.275" y2="38.735" width="0.6096" layer="1"/>
+<wire x1="43.18" y1="36.83" x2="45.72" y2="36.83" width="0.6096" layer="1"/>
+<wire x1="45.72" y1="36.83" x2="49.53" y2="33.02" width="0.6096" layer="1"/>
+<wire x1="49.53" y1="33.02" x2="49.53" y2="31.115" width="0.6096" layer="1"/>
 </signal>
 <signal name="N$3">
@@
 <contactref element="C21" pad="1"/>
 <contactref element="T1" pad="C"/>
-<wire x1="53.975" y1="36.83" x2="54.61" y2="36.195" width="0.6096" layer="16"/>
-<wire x1="54.61" y1="33.655" x2="54.61" y2="36.195" width="0.6096" layer="16"/>
 <wire x1="58.42" y1="33.655" x2="61.595" y2="36.83" width="0.6096" layer="16"/>
 <wire x1="61.595" y1="36.83" x2="63.5" y2="36.83" width="0.6096" layer="16"/>
@@
 <wire x1="67.31" y1="33.02" x2="67.31" y2="31.75" width="0.6096" layer="16"/>
 <wire x1="54.61" y1="33.655" x2="58.42" y2="33.655" width="0.6096" layer="16"/>
+<wire x1="51.435" y1="33.655" x2="54.61" y2="33.655" width="0.6096" layer="16"/>
 </signal>
 <signal name="N$52">
@@
 </board>
 </drawing>
+<compatibility>
+<note version="6.3" minversion="6.2.2" severity="warning">
+Since Version 6.2.2 text objects can contain more than one line,
+which will not be processed correctly with this version.
+</note>
+</compatibility>
 </eagle>
