File: psu_2.brd (EAGLE design)
At the start: 99.7 x 48.6 mm, 38 parts, among them IC1 7812TV

Commit message: Add files via upload
Parts:
- turned LED2 to 0 degrees
- turned LED4 to 180 degrees
Connections:
- net GND: now also LED2.A, LED4.A; no longer LED2.K, LED4.C
- net N$1: now also LED2.K, LED4.C; no longer LED2.A, LED4.A
Changed lines of the file:
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@@
 <attribute name="VALUE" x="80.01" y="28.321" size="1.27" layer="27" ratio="10" rot="R180"/>
 </element>
-<element name="LED2" library="led" package="LED3MM" value="" x="81.915" y="21.59" smashed="yes" rot="R180">
-<attribute name="NAME" x="79.629" y="20.32" size="1.016" layer="25" ratio="10" rot="R90"/>
-<attribute name="VALUE" x="80.01" y="23.241" size="1.27" layer="27" ratio="10" rot="R180"/>
+<element name="LED2" library="led" package="LED3MM" value="" x="81.915" y="21.59" smashed="yes">
+<attribute name="NAME" x="84.201" y="22.86" size="1.016" layer="25" ratio="10" rot="R270"/>
+<attribute name="VALUE" x="83.82" y="19.939" size="1.27" layer="27" ratio="10"/>
 </element>
 <element name="LED3" library="led" package="CHIPLED_1206" value="" x="86.995" y="27.94" smashed="yes" rot="R180">
@@
 <attribute name="VALUE" x="84.455" y="29.21" size="1.27" layer="27" rot="R270"/>
 </element>
-<element name="LED4" library="led" package="CHIPLED_1206" value="" x="86.995" y="20.32" smashed="yes">
-<attribute name="NAME" x="85.725" y="19.05" size="1.016" layer="25" rot="R90"/>
-<attribute name="VALUE" x="89.535" y="19.05" size="1.27" layer="27" rot="R90"/>
+<element name="LED4" library="led" package="CHIPLED_1206" value="" x="86.995" y="20.32" smashed="yes" rot="R180">
+<attribute name="NAME" x="88.265" y="21.59" size="1.016" layer="25" rot="R270"/>
+<attribute name="VALUE" x="84.455" y="21.59" size="1.27" layer="27" rot="R270"/>
 </element>
 <element name="ACIN" library="con-wago-508" package="W237-3E" value="" x="5.08" y="24.13" smashed="yes" rot="R90">
@@
 <contactref element="GND4" pad="1"/>
 <contactref element="GND1" pad="1"/>
-<contactref element="LED2" pad="K"/>
 <contactref element="LED1" pad="K"/>
-<contactref element="LED4" pad="C"/>
 <contactref element="LED3" pad="C"/>
 <contactref element="ACIN" pad="2"/>
@@
 <wire x1="92.71" y1="24.13" x2="95.25" y2="24.13" width="1.016" layer="16"/>
 <wire x1="80.645" y1="26.67" x2="80.645" y2="24.13" width="1.016" layer="16"/>
-<wire x1="80.645" y1="21.59" x2="80.645" y2="24.13" width="1.016" layer="16"/>
-<wire x1="86.995" y1="22.07" x2="86.995" y2="24.13" width="1.016" layer="1"/>
 <wire x1="86.995" y1="24.13" x2="92.71" y2="24.13" width="1.016" layer="1"/>
 <wire x1="86.995" y1="26.19" x2="86.995" y2="24.13" width="1.016" layer="1"/>
@@
 <wire x1="63.5" y1="35.56" x2="63.5" y2="24.13" width="1.016" layer="1"/>
 <wire x1="63.5" y1="24.13" x2="54.61" y2="24.13" width="1.016" layer="1"/>
+<contactref element="LED2" pad="A"/>
+<contactref element="LED4" pad="A"/>
+<wire x1="86.995" y1="22.07" x2="86.995" y2="24.13" width="1.016" layer="1"/>
+<wire x1="80.645" y1="24.13" x2="80.645" y2="21.59" width="1.016" layer="16"/>
 </signal>
 <signal name="N$3">
@@
 <signal name="N$1">
 <contactref element="R2" pad="1"/>
-<contactref element="LED4" pad="A"/>
-<contactref element="LED2" pad="A"/>
-<wire x1="83.185" y1="21.59" x2="84.455" y2="20.32" width="1.016" layer="1"/>
 <wire x1="84.455" y1="20.32" x2="84.455" y2="18.545" width="1.016" layer="1"/>
 <wire x1="84.455" y1="18.545" x2="86.97" y2="18.545" width="1.016" layer="1"/>
-<wire x1="86.97" y1="18.545" x2="86.995" y2="18.57" width="1.016" layer="1"/>
+<contactref element="LED4" pad="C"/>
+<contactref element="LED2" pad="K"/>
+<wire x1="86.995" y1="18.57" x2="86.97" y2="18.57" width="1.016" layer="1"/>
+<wire x1="86.97" y1="18.57" x2="86.97" y2="18.545" width="1.016" layer="1"/>
+<wire x1="83.185" y1="21.59" x2="84.455" y2="20.32" width="1.016" layer="1"/>
 </signal>
 <signal name="N$2">

Commit message: Add files via upload
Parts:
- removed +12V, +12V1, -12V, -12V1, GND1, GND2: (no value), wirepad:2,54/1,0
- added C1, C2, C3, C4: 1000u, rcl:E3,5-10
- C13, C17: device rcl:E3,5-8 -> rcl:E3,5-10
- moved C15 10.0 mm to (21.0, 14.6), turned to 270 degrees
- moved +12V3 8.25 mm to (83.8, 8.26)
- moved GND3 7.67 mm to (78.7, 8.26)
- moved +12V2 7.62 mm to (83.8, 39.4)
- moved -12V3 7.10 mm to (73.7, 8.26)
- moved GND4 6.98 mm to (78.7, 39.4)
- moved -12V2 6.35 mm to (73.7, 39.4)
- moved C10 1.42 mm to (26.0, 29.8)
- moved C13 1.42 mm to (23.5, 29.8)
- moved JP3 1.27 mm to (74.9, 24.1)
- moved JP1 1.27 mm to (34.3, 24.1)
- moved JP2 1.27 mm to (54.6, 24.1)
- moved JP4 1.27 mm to (95.2, 24.1)
- moved LED3 1.27 mm to (88.3, 27.9)
- moved LED4 1.27 mm to (88.3, 20.3)
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Connections:
- net +12V: now also C3.+; no longer +12V.1, +12V1.1
- net -12V: now also C4.-; no longer -12V.1, -12V1.1
- net GND: now also C1.-, C2.+, C3.-, C4.+; no longer GND1.1, GND2.1
- net N$3: now also C2.-
- net N$4: now also C1.+
Routing:
- net -12V: track 207.4 -> 143.0 mm
- net +12V: track 211.3 -> 150.9 mm
- net N$3: track 23.4 -> 68.0 mm
- net N$4: track 21.7 -> 58.4 mm
- net GND: track 275.1 -> 287.6 mm
- net N$1: track 6.14 -> 6.80 mm
- net N$2: track 6.12 -> 6.76 mm
