File: psu_2.sch (EAGLE design)
At the start: 32 parts, among them IC1 7812TV

Commit message: Add files via upload
Connections:
- net GND: now also LED2.A, LED4.A; no longer LED2.C, LED4.C
- net N$1: now also LED2.C, LED4.C; no longer LED2.A, LED4.A
Other:
- moved on the sheet: LED2, LED4
Changed lines of the file:
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@@
 <instance part="R2" gate="G$1" x="195.58" y="104.14" rot="R180"/>
 <instance part="LED1" gate="G$1" x="205.74" y="124.46"/>
-<instance part="LED2" gate="G$1" x="205.74" y="109.22" rot="R180"/>
+<instance part="LED2" gate="G$1" x="205.74" y="111.76"/>
 <instance part="LED3" gate="G$1" x="213.36" y="124.46"/>
-<instance part="LED4" gate="G$1" x="213.36" y="109.22" rot="R180"/>
+<instance part="LED4" gate="G$1" x="213.36" y="111.76"/>
 <instance part="ACIN" gate="-1" x="-22.86" y="139.7"/>
 <instance part="ACIN" gate="-2" x="-22.86" y="124.46"/>
@@
 <pinref part="GND1" gate="P" pin="P"/>
 <wire x1="91.44" y1="139.7" x2="91.44" y2="116.84" width="0.1524" layer="91"/>
-<pinref part="LED2" gate="G$1" pin="C"/>
 <pinref part="LED1" gate="G$1" pin="C"/>
-<wire x1="205.74" y1="114.3" x2="205.74" y2="116.84" width="0.1524" layer="91"/>
 <wire x1="205.74" y1="116.84" x2="205.74" y2="119.38" width="0.1524" layer="91"/>
 <wire x1="187.96" y1="116.84" x2="205.74" y2="116.84" width="0.1524" layer="91"/>
 <junction x="187.96" y="116.84"/>
 <junction x="205.74" y="116.84"/>
-<pinref part="LED4" gate="G$1" pin="C"/>
 <pinref part="LED3" gate="G$1" pin="C"/>
-<wire x1="213.36" y1="114.3" x2="213.36" y2="116.84" width="0.1524" layer="91"/>
 <wire x1="213.36" y1="116.84" x2="213.36" y2="119.38" width="0.1524" layer="91"/>
 <wire x1="205.74" y1="116.84" x2="213.36" y2="116.84" width="0.1524" layer="91"/>
+<pinref part="ACIN" gate="-2" pin="KL"/>
+<pinref part="LED2" gate="G$1" pin="A"/>
+<wire x1="205.74" y1="114.3" x2="205.74" y2="116.84" width="0.1524" layer="91"/>
+<pinref part="LED4" gate="G$1" pin="A"/>
+<wire x1="213.36" y1="114.3" x2="213.36" y2="116.84" width="0.1524" layer="91"/>
 <junction x="213.36" y="116.84"/>
-<pinref part="ACIN" gate="-2" pin="KL"/>
 </segment>
 </net>
@@
 <segment>
 <pinref part="R2" gate="G$1" pin="1"/>
-<pinref part="LED4" gate="G$1" pin="A"/>
 <wire x1="200.66" y1="104.14" x2="205.74" y2="104.14" width="0.1524" layer="91"/>
+<pinref part="LED4" gate="G$1" pin="C"/>
 <wire x1="205.74" y1="104.14" x2="213.36" y2="104.14" width="0.1524" layer="91"/>
 <wire x1="213.36" y1="104.14" x2="213.36" y2="106.68" width="0.1524" layer="91"/>
-<pinref part="LED2" gate="G$1" pin="A"/>
+<pinref part="LED2" gate="G$1" pin="C"/>
 <wire x1="205.74" y1="106.68" x2="205.74" y2="104.14" width="0.1524" layer="91"/>
 <junction x="205.74" y="104.14"/>

Commit message: Add files via upload
Parts:
- removed +12V, +12V1, -12V, -12V1, GND1, GND2: (no value), wirepad:2,54/1,0
- added C1, C2, C3, C4: 1000u, rcl:CPOL-EUE3.5-10
- C13, C17: device rcl:CPOL-EUE3.5-8 -> rcl:CPOL-EUE3.5-10
Connections:
- net +12V: now also C3.+; no longer +12V.P, +12V1.P
- net -12V: now also C4.-; no longer -12V.P, -12V1.P
- net GND: now also C1.-, C2.+, C3.-, C4.+; no longer GND1.P, GND2.P
- net N$3: now also C2.-
- net N$4: now also C1.+
Other:
- moved on the sheet: +12V2, +12V3, -12V2, -12V3, ACIN-1, ACIN-2, ACIN-3, B1, C10, C11, C13, C14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
