File: vc_reverb.brd (EAGLE design)
At the start: 99 x 49.8 mm, 90 parts, among them IC1 LM386N-1, IC2 LF411N, IC3 TL074P, IC4 LM13700N, IC5 TL072P, IC6 TL072P, T1 2N3906, T2 2N3906, X1 TOBU3, X2 TOBU3

Commit message: Add files via upload
Parts:
- moved C7 0.90 mm to (13.3, 8.89)
Routing:
- net GND: track 376.5 -> 377.4 mm
- net N$47: track 21.2 -> 20.6 mm
- added copper zone on layer 1, net GND
